File: Hardware/Macropad/USB.sch (KiCad schematic (older format))
At the start: 19 parts, among them J2 USB_C_Receptacle_USB2.0, U2 TCR2EF33, U3 SRV05-4

Commit message: Schematic mostly done. Started grouping components in layout
Parts:
- renumbered C17 to C1, C18 to C2, C19 to C3, J2 to J1, R10 to R1, R1 to R2, R9 to R3, R11 to R4, R12 to R5, R13 to R6, R14 to R7, R15 to R8, U2 to U1, U3 to U2
Other:
- moved on the sheet: C1, C2, C3, D1, FB1, FB2, FB3, J1, L1, R1, R2, R3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

Commit message: First pass of the layout done
Parts:
- removed R1: 1K, resistor_smd:R_0603_1608Metric, symbol Device:R
Connections:
- net +5V: now also U1.3 (CTRL)
- net D+: now also L1.2, R6.1, R8.2; no longer L1.1, R5.1, R7.2
- net D-: now also L1.1, R5.1, R7.2; no longer L1.2, R6.1, R8.2
- net at J1.A6 (D+), J1.B6 (D+), U2.3 (IO2): now also L1.3, R6.2; no longer L1.4, R5.2
- net at J1.A7 (D-), J1.B7 (D-), U2.1 (IO1): now also L1.4, R5.2; no longer L1.3, R6.2
- net USBD_N renamed USB_D0+
- net USBD_P renamed USB_D0-
Changed lines of the file:
@@
 L power:+5V #PWR01
 U 1 1 60D52A47
-P 1025 6800
+P 1025 7000
 AR Path="/6114D32E/60D52A47" Ref="#PWR01"  Part="1"
 AR Path="/6247A5CE/60D52A47" Ref="#PWR?"  Part="1"
-F 0 "#PWR01" H 1025 6650 50  0001 C CNN
-F 1 "+5V" H 1040 6973 50  0000 C CNN
-F 2 "" H 1025 6800 50  0001 C CNN
-F 3 "" H 1025 6800 50  0001 C CNN
-	1    1025 6800
+F 0 "#PWR01" H 1025 6850 50  0001 C CNN
+F 1 "+5V" H 1040 7173 50  0000 C CNN
+F 2 "" H 1025 7000 50  0001 C CNN
+F 3 "" H 1025 7000 50  0001 C CNN
+	1    1025 7000
 	1    0    0    -1
 $EndComp
@@
 	1825 7300 1775 7300
 $Comp
-L Device:R R1
-U 1 1 60D52A56
-P 875 7100
-AR Path="/6114D32E/60D52A56" Ref="R1"  Part="1"
-AR Path="/6247A5CE/60D52A56" Ref="R?"  Part="1"
-F 0 "R1" V 775 7100 50  0000 C CNN
-F 1 "1K" V 875 7100 50  0000 C CNN
-F 2 "resistor_smd:R_0603_1608Metric" V 805 7100 50  0001 C CNN
-F 3 "~" H 875 7100 50  0001 C CNN
-	1    875  7100
-	-1   0    0    1
-$EndComp
-Wire Wire Line
-	1025 6800 1025 6900
-Wire Wire Line
-	1075 7300 875  7300
-Wire Wire Line
-	875  6950 875  6900
-Wire Wire Line
-	875  6900 1025 6900
-Connection ~ 1025 6900
-Wire Wire Line
-	1025 6900 1025 7100
-$Comp
 L power:+3.3V #PWR04
 U 1 1 60D52A62
@@
 	1825 7100 1825 7025
 Wire Wire Line
-	875  7250 875  7300
-Wire Wire Line
 	4725 3125 4725 3175
 Wire Wire Line
@@
 Wire Wire Line
 	5525 2325 5625 2325
-Text GLabel 5625 2525 2    50   Output ~ 0
-USBD_N
-Text GLabel 5625 2325 2    50   Output ~ 0
-USBD_P
 $Comp
 L Device:R R7
@@
 	1625 3225 1625 3325
 Connection ~ 1625 3325
-Wire Wire Line
-	3975 2325 4200 2325
-Wire Wire Line
-	4200 2325 4200 2625
-Wire Wire Line
-	4200 2625 4475 2625
 Connection ~ 3975 2325
-Connection ~ 4475 2625
-Wire Wire Line
-	3850 2525 4325 2525
-Wire Wire Line
-	4325 2525 4325 2325
-Wire Wire Line
-	4325 2325 4475 2325
-Connection ~ 3850 2525
 Connection ~ 4475 2325
 Wire Wire Line
@@
 	4950 2525 5225 2525
 Text Label 5100 2325 0    50   ~ 0
+D-
+Text Label 5100 2525 0    50   ~ 0
 D+
-Text Label 5100 2525 0    50   ~ 0
-D-
 $Comp
 L Device:Ferrite_Bead FB3
@@
 Wire Notes Line
 	700  7625 700  6125
+Wire Wire Line
+	3850 2525 4475 2525
+Connection ~ 3850 2525
+Connection ~ 4475 2525
+Wire Wire Line
+	3975 2325 4475 2325
+Wire Wire Line
+	1075 7300 1025 7300
+Wire Wire Line
+	1025 7300 1025 7100
+Wire Wire Line
+	1025 7000 1025 7100
+Connection ~ 1025 7100
+Text GLabel 5625 2325 2    50   BiDi ~ 0
+USB_D0-
+Text GLabel 5625 2525 2    50   BiDi ~ 0
+USB_D0+
 $EndSCHEMATC

Commit message: Redoing layout with key switches upside down for better LED placement
Connections:
- net +5V: no longer FB3.1
- net GND: now also FB3.1
- net VBUS: no longer FB3.2
- net at C1.2, C2.2, FB1.2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: now also FB3.2
- net at J1.A6 (D+), J1.B6 (D+), L1.3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: now also U2.1 (IO1); no longer U2.3 (IO2)
- net at J1.A7 (D-), J1.B7 (D-), L1.4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: now also U2.6 (IO4); no longer U2.1 (IO1)
Other:
- moved on the sheet: FB3
Changed lines of the file:
@@
 L power:GND #PWR08
 U 1 1 60D529D7
-P 2775 3375
+P 2775 3825
 AR Path="/6114D32E/60D529D7" Ref="#PWR08"  Part="1"
 AR Path="/6247A5CE/60D529D7" Ref="#PWR?"  Part="1"
-F 0 "#PWR08" H 2775 3125 50  0001 C CNN
-F 1 "GND" H 2780 3202 50  0000 C CNN
-F 2 "" H 2775 3375 50  0001 C CNN
-F 3 "" H 2775 3375 50  0001 C CNN
-	1    2775 3375
+F 0 "#PWR08" H 2775 3575 50  0001 C CNN
+F 1 "GND" H 2780 3652 50  0000 C CNN
+F 2 "" H 2775 3825 50  0001 C CNN
+F 3 "" H 2775 3825 50  0001 C CNN
+	1    2775 3825
 	1    0    0    -1
 $EndComp
@@
 	2700 3325 2775 3325
 Wire Wire Line
-	2775 3325 2775 3375
-Wire Wire Line
 	2950 1775 3025 1775
 Wire Wire Line
@@
 	3050 2525 3850 2525
 Wire Wire Line
-	3975 2325 3975 3575
-Wire Wire Line
-	3975 3575 4225 3575
-Wire Wire Line
-	4225 3775 3850 3775
-Wire Wire Line
-	3850 3775 3850 2525
+	3975 2325 3975 2850
 NoConn ~ 5225 3575
-NoConn ~ 5225 3775
 Wire Wire Line
 	3875 1475 3875 1425
@@
 L Device:Ferrite_Bead FB3
 U 1 1 60DECA32
-P 3350 1525
+P 2525 3700
 AR Path="/6114D32E/60DECA32" Ref="FB3"  Part="1"
 AR Path="/6247A5CE/60DECA32" Ref="FB?"  Part="1"
-F 0 "FB3" V 3100 1425 50  0000 C CNN
-F 1 "Ferrite_Bead" V 3175 1450 50  0000 C CNN
-F 2 "Inductor_SMD:L_0805_2012Metric" V 3280 1525 50  0001 C CNN
-F 3 "~" H 3350 1525 50  0001 C CNN
-	1    3350 1525
+F 0 "FB3" V 2700 3700 50  0000 C CNN
+F 1 "Ferrite_Bead" V 2475 3100 50  0000 C CNN
+F 2 "Inductor_SMD:L_0805_2012Metric" V 2455 3700 50  0001 C CNN
+F 3 "~" H 2525 3700 50  0001 C CNN
+	1    2525 3700
 	0    1    1    0
 $EndComp
@@
 	1625 3325 2050 3325
 Wire Wire Line
-	2050 3325 2350 3325
+	2050 3325 2300 3325
 Connection ~ 2050 3325
 Wire Wire Line
@@
 Text GLabel 5625 2525 2    50   BiDi ~ 0
 USB_D0+
+Wire Wire Line
+	3975 2850 5375 2850
+Wire Wire Line
+	5375 2850 5375 3775
+Wire Wire Line
+	5375 3775 5225 3775
+Wire Wire Line
+	4225 3575 3850 3575
+Wire Wire Line
+	3850 3575 3850 2525
+NoConn ~ 4225 3775
+Wire Wire Line
+	2375 3700 2300 3700
+Wire Wire Line
+	2300 3700 2300 3325
+Connection ~ 2300 3325
+Wire Wire Line
+	2300 3325 2350 3325
+Wire Wire Line
+	2775 3325 2775 3700
+Wire Wire Line
+	2675 3700 2775 3700
+Connection ~ 2775 3700
+Wire Wire Line
+	2775 3700 2775 3825
 $EndSCHEMATC

Commit message: Layout done, cleaned up schematic and generated gerbers
Parts:
- added C16: 100nF, Capacitor_smd:C_0603_1608Metric, symbol Device:C
- added C30: 1uF, Capacitor_smd:C_0603_1608Metric, symbol Device:C
Connections:
- net +3V3: now also C30.1
- net +5V: now also C16.1
- net GND: now also C16.2, C30.2
Other:
- note added: "USB Upstream"
- note removed: "USB 2.0"
- moved on the sheet: C1, C2, C3, D1, FB1, FB2, FB3, J1, L1, R2, R3, R4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
