File: Hardware/Macropad/LEDs.sch (KiCad schematic (older format))
At the start: 58 parts

Commit message: Schematic mostly done. Started grouping components in layout
Parts:
- added D51: K40, custom_footprint_library:SK6812-MINI-E, symbol custom_parts_library:SK68XX-MINI-E
- added D52: K41, custom_footprint_library:SK6812-MINI-E, symbol custom_parts_library:SK68XX-MINI-E
- added D53: K42, custom_footprint_library:SK6812-MINI-E, symbol custom_parts_library:SK68XX-MINI-E
- added D54: K43, custom_footprint_library:SK6812-MINI-E, symbol custom_parts_library:SK68XX-MINI-E
- D23: renamed from D?; value UG_LED -> UG_LED_0; footprint custom_footprint_library:SK6812-MINI-E_0.4 -> custom_footprint_library:SK6812-MINI-E
- D24: renamed from D?; value UG_LED -> UG_LED_6; footprint custom_footprint_library:SK6812-MINI-E_0.4 -> custom_footprint_library:SK6812-MINI-E
- D25, D26, D27, D28, D31, D32, D33, D34, D37, D38, D39, D40, D43, D44, D45, D46: renamed from D?; footprint custom_footprint_library:SK6812-MINI-E_0.4 -> custom_footprint_library:SK6812-MINI-E
- D29: renamed from D?; value UG_LED -> UG_LED_1; footprint custom_footprint_library:SK6812-MINI-E_0.4 -> custom_footprint_library:SK6812-MINI-E
- D30: renamed from D?; value UG_LED -> UG_LED_7; footprint custom_footprint_library:SK6812-MINI-E_0.4 -> custom_footprint_library:SK6812-MINI-E
- D35: renamed from D?; value UG_LED -> UG_LED_2; footprint custom_footprint_library:SK6812-MINI-E_0.4 -> custom_footprint_library:SK6812-MINI-E
- D36: renamed from D?; value UG_LED -> UG_LED_8; footprint custom_footprint_library:SK6812-MINI-E_0.4 -> custom_footprint_library:SK6812-MINI-E
- D41: renamed from D?; value UG_LED -> UG_LED_3; footprint custom_footprint_library:SK6812-MINI-E_0.4 -> custom_footprint_library:SK6812-MINI-E
- D42: renamed from D?; value UG_LED -> UG_LED_9; footprint custom_footprint_library:SK6812-MINI-E_0.4 -> custom_footprint_library:SK6812-MINI-E
- D47: renamed from D?; value UG_LED -> UG_LED_4; footprint custom_footprint_library:SK6812-MINI-E_0.4 -> custom_footprint_library:SK6812-MINI-E
- D48: renamed from D?; value UG_LED -> UG_LED_10; footprint custom_footprint_library:SK6812-MINI-E_0.4 -> custom_footprint_library:SK6812-MINI-E
- D49: renamed from D?; value UG_LED -> UG_LED_5; footprint custom_footprint_library:SK6812-MINI-E_0.4 -> custom_footprint_library:SK6812-MINI-E
- D50: renamed from D?; value UG_LED -> UG_LED_11; footprint custom_footprint_library:SK6812-MINI-E_0.4 -> custom_footprint_library:SK6812-MINI-E
- gave numbers to parts that had none: 30
Connections:
- net +5V: now also D51.1 (VDD), D52.1 (VDD), D53.1 (VDD), D54.1 (VDD)
- net GND: now also D51.3 (GND), D52.3 (GND), D53.3 (GND), D54.3 (GND)
- net RGB[1]: now also D51.4 (DIN); no longer D25.4 (DIN)
- net at D25.2 (DOUT): now also D27.4 (DIN); no longer D31.4 (DIN)
- net at D31.2 (DOUT): now also D25.4 (DIN); no longer D37.4 (DIN)
- net at D43.2 (DOUT): now also D37.4 (DIN); no longer D45.4 (DIN)
- net at D37.2 (DOUT): now also D31.4 (DIN); no longer D43.4 (DIN)
- net at D45.2 (DOUT): now also D44.4 (DIN); no longer D39.4 (DIN)
- net at D39.2 (DOUT): now also D45.4 (DIN); no longer D33.4 (DIN)
- net at D27.2 (DOUT): now also D33.4 (DIN); no longer D26.4 (DIN)
- net at D33.2 (DOUT): now also D39.4 (DIN); no longer D27.4 (DIN)
- net at D26.2 (DOUT): now also D28.4 (DIN); no longer D32.4 (DIN)
- net at D32.2 (DOUT): now also D26.4 (DIN); no longer D38.4 (DIN)
- net at D44.2 (DOUT): now also D38.4 (DIN); no longer D46.4 (DIN)
- net at D38.2 (DOUT): now also D32.4 (DIN); no longer D44.4 (DIN)
- net at D46.2 (DOUT): now also R15.2; no longer D40.4 (DIN)
- net at D40.2 (DOUT): now also D46.4 (DIN); no longer D34.4 (DIN)
- net at D28.2 (DOUT): now also D34.4 (DIN); no longer R15.2
- net at D34.2 (DOUT): now also D40.4 (DIN); no longer D28.4 (DIN)
- new net: D43.4 (DIN), D54.2 (DOUT)
- new net: D53.2 (DOUT), D54.4 (DIN)
- new net: D52.2 (DOUT), D53.4 (DIN)
- new net: D51.2 (DOUT), D52.4 (DIN)
Other:
- note added: "LEDs"
- moved on the sheet: D23, D24, D25, D26, D27, D28, D29, D30, D31, D32, D33, D34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

Commit message: First pass of the layout done
Parts:
- removed C16, C30: 100nF, Capacitor_smd:C_0603_1608Metric, symbol Device:C
- removed D23: UG_LED_0, custom_footprint_library:SK6812-MINI-E, symbol custom_parts_library:SK68XX-MINI-E
- removed D29: UG_LED_1, custom_footprint_library:SK6812-MINI-E, symbol custom_parts_library:SK68XX-MINI-E
- added C40, C41, C42, C43: 100nF, Capacitor_smd:C_0603_1608Metric, symbol Device:C
Connections:
- net +5V: now also C40.1, C41.1, C42.1, C43.1
- net GND: now also C40.2, C41.2, C42.2, C43.2
- net at R16.2: now also D35.4 (DIN)
Other:
- moved on the sheet: R16

Commit message: Layout done, cleaned up schematic and generated gerbers
Other:
- moved on the sheet: C10, C11, C12, C13, C14, C15, C17, C18, C19, C20, C21, C22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

Commit message: Fixing a naming mistake in schematic
Parts:
- D24: value UG_LED_6 -> UG_LED_4
- D30: value UG_LED_7 -> UG_LED_5
- D35: value UG_LED_2 -> UG_LED_0
- D36: value UG_LED_8 -> UG_LED_6
- D41: value UG_LED_3 -> UG_LED_1
- D42: value UG_LED_9 -> UG_LED_7
- D47: value UG_LED_4 -> UG_LED_2
- D48: value UG_LED_10 -> UG_LED_8
- D49: value UG_LED_5 -> UG_LED_3
- D50: value UG_LED_11 -> UG_LED_9
Changed lines of the file:
@@
 AR Path="/61D5AB4C/61E450C6" Ref="D41"  Part="1"
 F 0 "D41" H 5025 1565 50  0000 C CNN
-F 1 "UG_LED_3" H 5025 1474 50  0000 C CNN
+F 1 "UG_LED_1" H 5025 1474 50  0000 C CNN
 F 2 "custom_footprint_library:SK6812-MINI-E" H 5000 1200 50  0001 C CNN
 F 3 "" H 5000 1200 50  0001 C CNN
@@
 AR Path="/61D5AB4C/61E48873" Ref="D35"  Part="1"
 F 0 "D35" H 4025 1565 50  0000 C CNN
-F 1 "UG_LED_2" H 4025 1474 50  0000 C CNN
+F 1 "UG_LED_0" H 4025 1474 50  0000 C CNN
 F 2 "custom_footprint_library:SK6812-MINI-E" H 4000 1200 50  0001 C CNN
 F 3 "" H 4000 1200 50  0001 C CNN
@@
 AR Path="/61D5AB4C/61E4C21D" Ref="D47"  Part="1"
 F 0 "D47" H 6025 1565 50  0000 C CNN
-F 1 "UG_LED_4" H 6025 1474 50  0000 C CNN
+F 1 "UG_LED_2" H 6025 1474 50  0000 C CNN
 F 2 "custom_footprint_library:SK6812-MINI-E" H 6000 1200 50  0001 C CNN
 F 3 "" H 6000 1200 50  0001 C CNN
@@
 AR Path="/61D5AB4C/61E4DC22" Ref="D49"  Part="1"
 F 0 "D49" H 7025 1565 50  0000 C CNN
-F 1 "UG_LED_5" H 7025 1474 50  0000 C CNN
+F 1 "UG_LED_3" H 7025 1474 50  0000 C CNN
 F 2 "custom_footprint_library:SK6812-MINI-E" H 7000 1200 50  0001 C CNN
 F 3 "" H 7000 1200 50  0001 C CNN
@@
 AR Path="/61D5AB4C/61E69B23" Ref="D24"  Part="1"
 F 0 "D24" H 2025 2590 50  0000 C CNN
-F 1 "UG_LED_6" H 2025 2499 50  0000 C CNN
+F 1 "UG_LED_4" H 2025 2499 50  0000 C CNN
 F 2 "custom_footprint_library:SK6812-MINI-E" H 2000 2225 50  0001 C CNN
 F 3 "" H 2000 2225 50  0001 C CNN
@@
 AR Path="/61D5AB4C/61E69B39" Ref="D30"  Part="1"
 F 0 "D30" H 3025 2590 50  0000 C CNN
-F 1 "UG_LED_7" H 3025 2499 50  0000 C CNN
+F 1 "UG_LED_5" H 3025 2499 50  0000 C CNN
 F 2 "custom_footprint_library:SK6812-MINI-E" H 3000 2225 50  0001 C CNN
 F 3 "" H 3000 2225 50  0001 C CNN
@@
 AR Path="/61D5AB4C/61E69B52" Ref="D42"  Part="1"
 F 0 "D42" H 5025 2590 50  0000 C CNN
-F 1 "UG_LED_9" H 5025 2499 50  0000 C CNN
+F 1 "UG_LED_7" H 5025 2499 50  0000 C CNN
 F 2 "custom_footprint_library:SK6812-MINI-E" H 5000 2225 50  0001 C CNN
 F 3 "" H 5000 2225 50  0001 C CNN
@@
 AR Path="/61D5AB4C/61E69B6B" Ref="D36"  Part="1"
 F 0 "D36" H 4025 2590 50  0000 C CNN
-F 1 "UG_LED_8" H 4025 2499 50  0000 C CNN
+F 1 "UG_LED_6" H 4025 2499 50  0000 C CNN
 F 2 "custom_footprint_library:SK6812-MINI-E" H 4000 2225 50  0001 C CNN
 F 3 "" H 4000 2225 50  0001 C CNN
@@
 AR Path="/61D5AB4C/61E69B84" Ref="D48"  Part="1"
 F 0 "D48" H 6025 2590 50  0000 C CNN
-F 1 "UG_LED_10" H 6025 2499 50  0000 C CNN
+F 1 "UG_LED_8" H 6025 2499 50  0000 C CNN
 F 2 "custom_footprint_library:SK6812-MINI-E" H 6000 2225 50  0001 C CNN
 F 3 "" H 6000 2225 50  0001 C CNN
@@
 AR Path="/61D5AB4C/61E69B9D" Ref="D50"  Part="1"
 F 0 "D50" H 7025 2590 50  0000 C CNN
-F 1 "UG_LED_11" H 7025 2499 50  0000 C CNN
+F 1 "UG_LED_9" H 7025 2499 50  0000 C CNN
 F 2 "custom_footprint_library:SK6812-MINI-E" H 7000 2225 50  0001 C CNN
 F 3 "" H 7000 2225 50  0001 C CNN
