File: Hardware/Macropad/Macropad.kicad_pcb (KiCad board)
At the start: 2 copper layers, 89 x 130.9 mm, 172 parts, among them J1 USB_C_Receptacle_USB2.0, J2 Conn_01x04_Female, J3 Conn_02x03_Odd_Even, J4 USB_C_Receptacle_USB2.0, J5 USB_C_Receptacle_USB2.0, J6 USB_C_Receptacle_USB2.0, SW1 K40_1U, SW10 K01_1U, SW11 K42_1U, SW12 K32_1U, SW13 K22_1U, SW14 K12_1U, SW15 K02_1U, SW16 K43_1U, SW17 K33_1U, SW18 K23_1U, SW19 K13_1U, SW2 K30_1U, SW20 K03_1U, SW21 Rotary_Encoder_Switch, SW22 SW_Push, SW3 K20_1U, SW4 K10_1U, SW5 K00_1U, SW6 K41_1U, SW7 K31_1U, SW8 K21_1U, SW9 K11_1U, U1 TCR2EF33, U2 SRV05-4, U4 TUSB2046b, U5 ATmega32U4-AU, U6 SRV05-4, U8 SRV05-4, X1 KC2016K, X2 625L3C006M00000

Commit message: Fixing a naming mistake in schematic
Parts:
- D24: value UG_LED_6 -> UG_LED_4
- D30: value UG_LED_7 -> UG_LED_5
- D35: value UG_LED_2 -> UG_LED_0
- D36: value UG_LED_8 -> UG_LED_6
- D41: value UG_LED_3 -> UG_LED_1
- D42: value UG_LED_9 -> UG_LED_7
- D47: value UG_LED_4 -> UG_LED_2
- D48: value UG_LED_10 -> UG_LED_8
- D49: value UG_LED_5 -> UG_LED_3
- D50: value UG_LED_11 -> UG_LED_9
